Commit message: urdf change3

File: src/robotv1_description/urdf/robot_1.urdf (robot description, URDF)
Before this commit: robot my_robot, 1 links, 0 joints
Links:
- added link base_link; collision mesh filename=package://robotv1_description/meshes/base_link.stl; visual mesh filename=package://robotv1_description/meshes/base_link.stl
- link base: geometry collision mesh filename=package://robotv1_description/meshes/base.stl; visual mesh filename=package://robotv1_description/meshes/base.stl
Joints:
- added joint base_to_base_link: type revolute, parent base, child base_link, origin xyz=0 0 0 rpy=0 0 0, axis 0 0 1, limit lower=-1.57 upper=1.57 effort=5 velocity=1

Commit message: final urdf

File: src/robotv1_description/urdf/robot_1.urdf (robot description, URDF)
Before this commit: robot my_robot, 2 links, 1 joints
Links:
- added link radar_link; visual mesh filename=package://robotv1_description/meshes/radar_link.stl
- added link shoulder; visual mesh filename=package://robotv1_description/meshes/shoulder_link.stl
- link base: geometry collision box size=0.12 0.12 0.05; visual mesh filename=package://robotv1_description/meshes/base.stl
- link base_link: geometry collision box size=0.04 0.12 0.05; visual mesh filename=package://robotv1_description/meshes/base_link.stl
Joints:
- added joint radar_to_shoulder: type revolute, parent shoulder, child radar_link, origin xyz=0.099733 0 0.089263 rpy=0 0 0, axis 0 1 0, limit lower=-1.57 upper=1.57 effort=5 velocity=1
- added joint shouler_to_base: type revolute, parent base_link, child shoulder, origin xyz=0 0 0.115430 rpy=0 0 0, axis 0 1 0, limit lower=-2.424 upper=0.7173303 effort=5 velocity=1
- joint base_to_base_link: limit lower=-1.57 upper=1.57 effort=5 velocity=1 -> (none); type revolute -> continuous

Commit message: m

File: src/robotv1_description/urdf/robot_1.urdf (robot description, URDF)
Before this commit: robot my_robot, 4 links, 3 joints
Links:
- link base: geometry collision mesh filename=package://robotv1_description/meshes/base.stl; visual mesh filename=package://robotv1_description/meshes/base.stl
- link base_link: mass None -> 1; geometry collision mesh filename=package://robotv1_description/meshes/base_link.stl; visual mesh filename=package://robotv1_description/meshes/base_link.stl
- link shoulder: geometry visual mesh filename=package://robotv1_description/meshes/rod_shaft.stl

Commit message: change

File: src/robotv1_description/urdf/robot_1.urdf (robot description, URDF)
Before this commit: robot my_robot, 4 links, 3 joints
Links:
- link radar_link: mass None -> 0.5; geometry collision mesh filename=package://robotv1_description/meshes/radar_link.stl; visual mesh filename=package://robotv1_description/meshes/radar_link.stl
- link shoulder: mass None -> 0.5; geometry collision mesh filename=package://robotv1_description/meshes/rod_shaft.stl; visual mesh filename=package://robotv1_description/meshes/rod_shaft.stl

Commit message: changes

File: src/robotv1_description/urdf/robot_1.urdf (robot description, URDF)
Before this commit: robot my_robot, 4 links, 3 joints
Links:
- link base: mass 2 -> 0.72
- link base_link: mass 1 -> 1.25
